Commit message: hardware testing 27-8 1

File: quad_simulator/jamal_description/urdf/jamal_tested.urdf (robot description, URDF)
Before this commit: robot jamal_description, 24 links, 23 joints
Links:
- added link odom
- added link t265_link
Joints:
- removed joint base_static_joint
- added joint map_to_odom: type fixed, parent map, child odom, origin xyz=0 0 0 rpy=0 0 0
- added joint odom_to_base: type fixed, parent odom, child body, origin xyz=0 0 0 rpy=0 0 0
- added joint t265_joint: type fixed, parent trunk, child t265_link, origin xyz=0.175 0 0.08 rpy=0 0 0
- joint floating_base: origin xyz=0 0 0 rpy=0 0 0 -> xyz=0 0 0.07 rpy=0 0 0
