Commit message: HW Testing 27-10 2

File: quad_simulator/jamal_description/urdf/jamal_tested_sim.urdf (robot description, URDF)
Before this commit: robot jamal_description, 26 links, 25 joints
Joints:
- joint map_to_odom: origin xyz=0 0 0 rpy=0 0 0 -> xyz=0 0 0.0665 rpy=0 0 0
- joint t265_joint: origin xyz=0.175 0 0.08 rpy=0 0 0 -> xyz=0.175 0 0.08 rpy=0 0.08 0
